File: kicad/stm32-main/screen.kicad_sch (KiCad schematic)
At the start: 1 part, among them J7 DO0180FMST03

Commit message: hw: screen updates
Parts:
- added C11, C8, C9: 10uF, symbol Device:C
Connections:
- net GND: now also C11.2, C8.2, C9.2
- net VBAT: now also C11.1
- net TP_RST: now reaches J7.14 (Pin_14)
- net +3.3V: now reaches J7.16 (Pin_16)
- net +3.3V: now also J7.17 (Pin_17), J7.24 (Pin_24), J7.26 (Pin_26), C8.1, C9.1
- removed net PWR: J7.17 (Pin_17), J7.22 (Pin_22), J7.26 (Pin_26)
- new net PWR_EN: J7.22 (Pin_22)
- no-connect marks 6 -> 5
Other:
- note added: "TP_VCC 2.7V - 3.4V"
- note added: "VBAT typ. 3.8V (2.9-4.5V)"
- note added: "VCI 2.7V - 3.6V"
- note removed: "Note: 2.7V - 3.6V"
- note removed: "Note: 2.8V - 3.4V"
- note removed: "Share a 2.8V LDO? Battery shouldn't go below this voltage"
