File: kicad/stm32-main/power-control-i2c.kicad_sch (KiCad schematic)
At the start: 1 part, among them IC4 BQ25628ERYKR

Commit message: hw: add bq25628e rough design
Parts:
- added BT2: Battery_Cell, symbol Device:Battery_Cell
- added C12: 47nF, symbol Device:C
- added C13: 4.7uF, symbol Device:C
- added C14, C15: 10uF, symbol Device:C
- added L1: 1uH, symbol Device:L
- added R6, R7, R8: R, symbol Device:R
Connections:
- net SCL: now also IC4.13 (SCL)
- net SDA: now also IC4.12 (SDA)
- net ~{BAT_INT}: now also IC4.11 (~{INT})
- net ~{PG}: now also IC4.3 (~{PG})
- net BTST: now reaches IC4.1 (BTST_1)
- net BTST: now also C12.2
- net STAT: now reaches IC4.10 (STAT_1)
- net CE: now reaches IC4.14 (~{CE_1})
- net GND: now reaches IC4.15 (GND)
- net GND: now also BT2.2 (-), C13.2, C14.2, C15.2, R6.2, R8.2
- net SW: now reaches IC4.16 (SW)
- net SW: now also C12.1, L1.1
- net PMID: now reaches IC4.17 (PMID)
- net PMID: now also C15.1
- net VBUS: now reaches IC4.18 (VBUS)
- net VBUS: now also C14.1
- net REGN: now reaches IC4.2 (REGN)
- net REGN: now also C13.1
- net ~{CE}: now reaches IC4.22 (~{CE_2})
- net ILIM: now reaches IC4.4 (ILIM)
- net ILIM: now also R6.1
- net TS_BIAS: now reaches IC4.5 (TS_BIAS_1)
- net TS_BIAS: now also R7.1
- net TS: now reaches IC4.6 (TS)
- net TS: now also R7.2, R8.1
- net BAT: now reaches IC4.8 (BAT)
- net BAT: now also BT2.1 (+)
- net VSYS: now reaches IC4.9 (SYS)
- net VSYS: now also L1.2
- no-connect marks 0 -> 4
Other:
- note added: "Bat doesn't have thermistor Assuming hard-wiring will be fine"
- note added: "Ceramic!"
- note added: "Ceramic! As close to pins as possible"
- note added: "Exit ship mode/chip reset"
- note added: "LOW=on charge, blinks 1Hz on fault Leave floating if unused"
- note added: "Rec. 10k resistor for pull-ups"
- note added: "_Charge_ enable MUST be driven"
