File: kicad/pico2-carrier/screen-headers.kicad_sch (KiCad schematic)
At the start: 11 parts, among them J1 SCREEN_HDR, J2 TP_HDR, J3 Ext_Pwr_Rail, J4 DO0180FMST08

Commit message: hw: lots of changes to pico 2 board
Parts:
- removed C8: 10uF, Capacitor_SMD:C_0402_1005Metric, symbol Device:C
- removed J2: TP_HDR, symbol Connector_Generic:Conn_01x04
- removed R4: 0R, Resistor_SMD:R_0805_2012Metric, symbol Device:R
- J2: renamed from J1; footprint (none) -> Connector_PinHeader_2.54mm:PinHeader_1x08_P2.54mm_Vertical
- J3: renamed from J4; footprint AXE534127 -> SamacsysParts:AXE534127
- J5: renamed from J3; footprint Connector_PinHeader_2.54mm:PinHeader_2x06_P2.54mm_Vertical -> Connector_PinHeader_2.54mm:PinHeader_2x07_P2.54mm_Vertical; symbol Connector_Generic:Conn_02x06_Counter_Clockwise -> Connector_Generic:Conn_02x07_Odd_Even
- JP3: renamed from JP1; footprint (none) -> Jumper:SolderJumper-3_P1.3mm_Open_Pad1.0x1.5mm
- JP4: renamed from JP2; footprint (none) -> Jumper:SolderJumper-3_P1.3mm_Open_Pad1.0x1.5mm
- renumbered C10 to C8
Connections:
- net +3.3V: now also J5.14 (Pin_14), J5.2 (Pin_2), J5.4 (Pin_4), J5.6 (Pin_6); no longer J5.11 (Pin_11), J5.7 (Pin_7), J5.9 (Pin_9)
- net GND: now also J5.11 (Pin_11), J5.13 (Pin_13), J5.7 (Pin_7), J5.9 (Pin_9); no longer J5.2 (Pin_2), J5.4 (Pin_4), J5.6 (Pin_6)
- net TP_VCC: now reaches J3.16 (TP_VCC)
- net TE: now reaches J3.2 (TE)
- net VPP: now reaches J3.34 (VPP)
- no-connect marks 9 -> 14
Other:
- note added: "Needs to be 12.0mm from edge of board, odds side facing edge"
- moved on the sheet: C8, C9
